File: jalapeno.kicad_pcb (KiCad board)
At the start: 2 copper layers, 233.4 x 81 mm, 133 parts, among them IC1 ATMEGA32U4-AU, J1 USB_B, J2 AVR-ISP-6, J3 Conn_01x04, K1 esc, K10 o, K11 p, K12 back, K13 tab, K14 a, K15 s, K16 d, K17 f, K18 g, K19 h, K2 q, K20 j, K21 k, K22 l, K23 ;, K24 caps, K25 caps, K26 z, K27 x, K28 c, K29 v, K3 w, K30 b, K31 n, K32 m, K33 ,, K33_1 ,, K34 ., K34_1 ., K35 ctrl, K36 gui, K37 alt, K37_1 alt, K38 space, K38_1 space, K39 alt, K39_1 gui, K4 e, K40 gui, K41 ctrl, K42 KEYSW, K5 r, K6 t, K7 y, K8 u, K9 i, SW1 SW_PUSH, U1 MDBT40, U2 SPX3819M5-L-3-3, U3 MCP73831T-2ACI/OT, Y1 XTAL_GND

Commit message: gerber export & logo
Parts:
- added G***: LOGO, Jalapeno:LOGO_MASK, F.Cu at (73.6, 98.6)
Routing:
- net GND: track 33.3 -> 37.9 mm
Other:
- board text added: "BLE"
- board text added: "V0.0.2"

Commit message: v0.3.0
Parts:
- removed G***: LOGO, Jalapeno:LOGO_MASK
- removed H5: MountingHole_2.2mm_M2_Pad, Mounting_Holes:MountingHole_2.2mm_M2_Pad
- added G1: Mounting_Hole, Jalapeno:LOGO, B.Cu at (104.8, 90.8)
- added G1_0: Mounting_Hole, Jalapeno:LOGO, F.Cu at (104.8, 90.8)
- added G2: Mounting_Hole, Jalapeno:OSHW_Logo, B.Cu at (234.1, 56.6)
- added G3: Mounting_Hole, Jalapeno:CC-BY-NC-SA, B.Cu at (231.2, 61.1)
- H1, H2, H3, H4, H6: value MountingHole_2.2mm_M2_Pad -> Mounting_Hole
- K38: footprint Jalapeno:CHERRY_PCB_625H_NO_BORDER -> Jalapeno:CHERRY_PCB_625H_NO_BORDER_FLIP_STAB
- K38_1: footprint Jalapeno:CHERRY_PCB_225H_NO_BORDER -> Jalapeno:CHERRY_PCB_225H_NO_BORDER_FLIP_STAB
- K42: footprint Jalapeno:CHERRY_PCB_275H_NO_BORDER -> Jalapeno:CHERRY_PCB_275H_NO_BORDER_FLIP_STAB
- moved J2 50.2 mm to (173.8, 98.0)
- moved D42 2.75 mm to (165.1, 92.8)
- moved U1 1.80 mm to (142.0, 91.6)
- moved J1 1.79 mm to (147.6, 29.2)
- moved LED1_0 1.79 mm to (33.8, 76.0)
- moved LED2_0 1.79 mm to (33.8, 81.0)
- moved R1 1.79 mm to (35.8, 81.0)
- moved R2 1.79 mm to (35.8, 76.0)
- moved J3 1.64 mm to (35.2, 61.9)
- moved D41 0.79 mm to (203.6, 94.6)
Routing:
- net VBUS: track 493.4 -> 412.5 mm, vias 23 -> 19
- net /RESET: track 219.7 -> 187.0 mm, vias 11 -> 8
- net ROW_1: track 323.2 -> 350.8 mm
- net /MOSI: track 66.3 -> 57.4 mm, vias 2 -> 3
- net /SCK: track 70.3 -> 62.8 mm
- net /MISO: track 65.9 -> 59.6 mm, vias 2 -> 3
- net /4_SWDIO/RST: track 258.8 -> 254.8 mm, vias 7 -> 9
- net GND: track 37.9 -> 34.3 mm
- net /SWDCLK: track 151.7 -> 148.1 mm
- net Net-(R2-Pad1): track 207.8 -> 206.0 mm
- net Net-(J1-Pad3): track 6.58 -> 4.80 mm
- net ROW_4: track 217.7 -> 219.5 mm
- net /8_BLE_CS: track 81.8 -> 80.1 mm
- net /7_BLE_IRQ: track 108.1 -> 106.4 mm
- net Net-(D42-Pad2): track 7.95 -> 6.38 mm
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Other:
- board size 233.4 x 81 mm -> 230.1 x 77.6 mm
- board text added: "+"
- board text added: "."
- board text added: "CLK"
- board text added: "DIO"
- board text added: "GND"
- board text added: "MISO"
- board text added: "MOSI"
- board text added: "RESET"
- board text added: "RST"
- board text added: "SCK"
- board text added: "VBUS"
- board text added: "open source hardware"
- board text added: "v0.3"
- board text added: "©2018 geewizwow"
- board text removed: "BLE"
- board text removed: "KEEPOUT"
- board text removed: "V0.0.2"

Commit message: logos
Parts:
- added G4: Copyright, Jalapeno:COPYRIGHT, B.Cu at (43.9, 99.3)
- G1: value Mounting_Hole -> Logo
- G1_0: value Mounting_Hole -> Logo Front
- G2: value Mounting_Hole -> OSHW logo
- G3: value Mounting_Hole -> CC logo
Other:
- board text added: "JLCJLCJL-CJ-LCJLCJ"
- board text removed: "©2018 geewizwow"

Commit message: rgb caps
Parts:
- added CR1: 0.1uf, Capacitors_SMD:C_0805_HandSoldering, B.Cu at (77.1, 81.0)
- added CR2: 0.1uf, Capacitors_SMD:C_0805_HandSoldering, B.Cu at (129.1, 81.0)
- added CR3: 0.1uf, Capacitors_SMD:C_0805_HandSoldering, B.Cu at (166.1, 81.0)
- added CR4: 0.1uf, Capacitors_SMD:C_0805_HandSoldering, B.Cu at (229.0, 81.0)
- added CR5: 0.1uf, Capacitors_SMD:C_0805_HandSoldering, B.Cu at (218.2, 42.9)
- added CR6: 0.1uf, Capacitors_SMD:C_0805_HandSoldering, B.Cu at (166.1, 42.9)
- added CR7: 0.1uf, Capacitors_SMD:C_0805_HandSoldering, B.Cu at (118.6, 42.9)
- added CR8: 0.1uf, Capacitors_SMD:C_0805_HandSoldering, B.Cu at (76.6, 42.9)
Routing:
- net +3V3: track 607.7 -> 637.2 mm, vias 20 -> 21
Other:
- net class Default: trace_width 0.15 -> 0.2

Commit message: placed components
Parts:
- removed R10: 10k, Resistors_SMD:R_0805_HandSoldering
- added Q1: MMBT2222ALT3G, TO_SOT_Packages_SMD:SOT-23, B.Cu at (142.2, 119.5)
- added RK1: 330, Jalapeno:R_0805, B.Cu at (37.8, 30.1)
- added RK10: 330, Jalapeno:R_0805, B.Cu at (209.3, 30.1)
- added RK11: 330, Jalapeno:R_0805, B.Cu at (228.3, 30.1)
- added RK12: 330, Jalapeno:R_0805, B.Cu at (247.4, 29.8)
- added RK13: 330, Jalapeno:R_0805, B.Cu at (40.2, 49.1)
- added RK14: 330, Jalapeno:R_0805, B.Cu at (61.6, 49.1)
- added RK15: 330, Jalapeno:R_0805, B.Cu at (80.7, 49.1)
- added RK16: 330, Jalapeno:R_0805, B.Cu at (99.7, 49.1)
- added RK17: 330, Jalapeno:R_0805, B.Cu at (118.8, 49.1)
- added RK18: 330, Jalapeno:R_0805, B.Cu at (137.8, 49.1)
- added RK19: 330, Jalapeno:R_0805, B.Cu at (156.9, 49.1)
- added RK2: 330, Jalapeno:R_0805, B.Cu at (56.9, 30.1)
- added RK20: 330, Jalapeno:R_0805, B.Cu at (175.9, 49.1)
- added RK21: 330, Jalapeno:R_0805, B.Cu at (195.0, 49.1)
- added RK22: 330, Jalapeno:R_0805, B.Cu at (214.0, 49.1)
- added RK23: 330, Jalapeno:R_0805, B.Cu at (240.2, 49.1)
- added RK24: 330, Jalapeno:R_0805, B.Cu at (44.9, 68.2)
- added RK25: 330, Jalapeno:R_0805, B.Cu at (71.1, 68.2)
- added RK26: 330, Jalapeno:R_0805, B.Cu at (90.2, 68.2)
- added RK27: 330, Jalapeno:R_0805, B.Cu at (109.2, 68.2)
- added RK28: 330, Jalapeno:R_0805, B.Cu at (128.3, 68.2)
- added RK29: 330, Jalapeno:R_0805, B.Cu at (147.3, 68.2)
- added RK30: 330, Jalapeno:R_0805, B.Cu at (166.4, 68.2)
- added RK31: 330, Jalapeno:R_0805, B.Cu at (185.4, 68.2)
- added RK32: 330, Jalapeno:R_0805, B.Cu at (204.5, 68.2)
- added RK33: 330, Jalapeno:R_0805, B.Cu at (223.5, 68.2)
- added RK34: 330, Jalapeno:R_0805, B.Cu at (245.0, 68.2)
- added RK35: 330, Jalapeno:R_0805, B.Cu at (40.2, 87.2)
- added RK36: 330, Jalapeno:R_0805, B.Cu at (61.6, 87.2)
- added RK37: 330, Jalapeno:R_0805, B.Cu at (80.7, 87.2)
- added RK38: 330, Jalapeno:R_0805, B.Cu at (149.7, 87.2)
- added RK39: 330, Jalapeno:R_0805, B.Cu at (221.2, 87.2)
- added RK4: 330, Jalapeno:R_0805, B.Cu at (95.0, 30.1)
- added RK40: 330, Jalapeno:R_0805, B.Cu at (245.0, 87.2)
- added RK41: 330, Jalapeno:R_0805, B.Cu at (202.1, 87.2)
- added RK42: 330, Jalapeno:R_0805, B.Cu at (164.0, 87.2)
- added RK5: 330, Jalapeno:R_0805, B.Cu at (114.0, 30.1)
- added RK6: 330, Jalapeno:R_0805, B.Cu at (133.1, 30.1)
- added RK7: 330, Jalapeno:R_0805, B.Cu at (153.6, 30.1)
- added RK8: 330, Jalapeno:R_0805, B.Cu at (171.2, 30.1)
- added RK9: 330, Jalapeno:R_0805, B.Cu at (190.2, 30.1)
- added Rk3: 330, Jalapeno:R_0805, B.Cu at (75.9, 30.1)
- C1, C2, C3, C4, C5, C6, C7, CR1, CR2, CR3, CR4, CR5, CR6, CR7, CR8: footprint Capacitors_SMD:C_0805_HandSoldering -> Capacitors_SMD:C_0805
- D1, D10, D11, D12, D13, D14, D15, D16, D17, D18, D19, D2, D20, D21, D22, D23, D24, D25, D26, D27, D28, D29, D3, D30, D31, D32, D33, D34, D35, D36, D37, D38, D39, D4, D40, D41, D42, D5, D6, D7, D8, D9: footprint Diodes_SMD:D_0805 -> Jalapeno:D_0805
- K1, K10, K11, K12, K14, K15, K16, K17, K18, K19, K2, K20, K21, K22, K25, K26, K27, K28, K29, K3, K30, K31, K32, K33_1, K36, K37, K4, K5, K6, K7, K8, K9: footprint Jalapeno:CHERRY_PCB_100H_NO_BORDER -> Jalapeno:CHERRY_PCB_100H_LED
- K13, K34_1, K35, K39, K40, K41: footprint Jalapeno:CHERRY_PCB_125H_NO_BORDER -> Jalapeno:CHERRY_PCB_125H_LED
- K23, K24: footprint Jalapeno:CHERRY_PCB_175H_NO_BORDER -> Jalapeno:CHERRY_PCB_175H_LED
- K33, K37_1: footprint Jalapeno:CHERRY_PCB_125H_NO_BORDER -> Jalapeno:CHERRY_PCB_125H_LED_REVERSED
- K34, K39_1: footprint Jalapeno:CHERRY_PCB_100H_NO_BORDER -> Jalapeno:CHERRY_PCB_100H_LED_REVERSED
- K38: footprint Jalapeno:CHERRY_PCB_625H_NO_BORDER_FLIP_STAB -> Jalapeno:CHERRY_PCB_625H_LED
- K38_1: footprint Jalapeno:CHERRY_PCB_225H_NO_BORDER_FLIP_STAB -> Jalapeno:CHERRY_PCB_225H_LED
- K42: footprint Jalapeno:CHERRY_PCB_275H_NO_BORDER_FLIP_STAB -> Jalapeno:CHERRY_PCB_275H_LED
- R1, R2, R4, R5, R6, R8: footprint Resistors_SMD:R_0805_HandSoldering -> Resistors_SMD:R_0805
- R3, R7: value 100k -> 10k; footprint Resistors_SMD:R_0805_HandSoldering -> Resistors_SMD:R_0805
- R9: value 10k -> 1.5k; footprint Resistors_SMD:R_0805_HandSoldering -> Resistors_SMD:R_0805
- moved R6 102.0 mm to (120.0, 115.2)
- moved R9 101.3 mm to (142.1, 125.8)
- moved JST1 84.8 mm to (176.2, 131.0)
- moved C3 71.4 mm to (207.5, 121.7)
- moved U3 71.4 mm to (207.5, 117.9)
- moved R7 70.1 mm to (63.3, 62.0), turned to 180 degrees
- moved U2 62.9 mm to (120.0, 118.5)
- moved C5 62.4 mm to (120.0, 122.6)
- moved C6 62.4 mm to (117.9, 122.6)
- moved C7 62.4 mm to (122.0, 122.6)
- moved DB1 62.2 mm to (186.3, 123.5)
- moved R3 56.1 mm to (207.5, 114.0), turned to 0 degrees
- moved D38 43.5 mm to (159.8, 86.0), turned to 270 degrees
- moved R8 42.2 mm to (198.4, 83.5), turned to 90 degrees
- moved D33 14.9 mm to (236.0, 67.0), turned to 270 degrees
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Connections:
- IC1 pad 29: /BATT_LVL -> LEDPWM
- R3 pad 1: /BATT_LVL -> GND
- R3 pad 2: +BATT -> Net-(R3-Pad2)
- R6 pad 1: GND -> Net-(R6-Pad1)
- R6 pad 2: /BATT_LVL -> VBUS
- R7 pad 1: Net-(R7-Pad1) -> +3V3
- R7 pad 2: VBUS -> /RESET
- R8 pad 1: GND -> Net-(IC1-Pad33)
- R8 pad 2: Net-(R8-Pad2) -> GND
- R9 pad 1: +3V3 -> Net-(Q1-Pad1)
- R9 pad 2: /RESET -> LEDPWM
- U2 pad 3: Net-(R7-Pad1) -> Net-(R6-Pad1)
- U3 pad 5: Net-(R8-Pad2) -> Net-(R3-Pad2)
Routing:
- net +3V3: track 637.2 -> 0.00 mm, vias 21 -> 0
- net VBUS: track 412.5 -> 0.00 mm, vias 19 -> 0
- net ROW_1: track 350.8 -> 0.00 mm, vias 17 -> 0
- net COL_1: track 260.0 -> 0.00 mm, vias 7 -> 0
- net ROW_2: track 255.9 -> 0.00 mm, vias 12 -> 0
- net /4_SWDIO/RST: track 254.8 -> 0.00 mm, vias 9 -> 0
- net ROW_3: track 235.7 -> 0.00 mm, vias 12 -> 0
- net COL_4: track 228.0 -> 0.00 mm, vias 5 -> 0
- net COL_2: track 223.9 -> 0.00 mm, vias 9 -> 0
- net ROW_4: track 219.5 -> 0.00 mm, vias 9 -> 0
- net COL_6: track 218.8 -> 0.00 mm, vias 7 -> 0
- net COL_3: track 215.9 -> 0.00 mm, vias 5 -> 0
- net Net-(R2-Pad1): track 206.0 -> 0.00 mm, vias 4 -> 0
- net COL_5: track 193.3 -> 0.00 mm, vias 6 -> 0
- net /RESET: track 187.0 -> 0.00 mm, vias 8 -> 0
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Other:
- net class Default: trace_width 0.2 -> 0.15
- board text added: "v0.4"
- board text removed: "v0.3"

Commit message: routing + plate
Parts:
- H1, H2, H3, H4, H6: footprint Mounting_Holes:MountingHole_2.2mm_M2_Pad -> Jalapeno:NOOP
- K33, K37_1: footprint Jalapeno:CHERRY_PCB_125H_LED_REVERSED -> Jalapeno:CHERRY_PCB_125H_LED
- K33_1, K37: footprint Jalapeno:CHERRY_PCB_100H_LED -> Jalapeno:CHERRY_PCB_100H_LED_REVERSED
- K34, K39_1: footprint Jalapeno:CHERRY_PCB_100H_LED_REVERSED -> Jalapeno:CHERRY_PCB_100H_LED
- K34_1, K39: footprint Jalapeno:CHERRY_PCB_125H_LED -> Jalapeno:CHERRY_PCB_125H_LED_REVERSED
- moved JST1 92.8 mm to (204.8, 42.7)
- moved C3 80.4 mm to (194.4, 42.4), turned to 90 degrees
- moved DB1 78.1 mm to (190.5, 45.5), turned to 0 degrees
- moved U3 77.3 mm to (190.5, 42.4), turned to 180 degrees
- moved R3 74.6 mm to (186.6, 42.4), turned to 90 degrees
- moved R6 68.9 mm to (133.3, 47.6)
- moved U2 67.4 mm to (133.3, 52.4)
- moved C5 67.3 mm to (133.3, 56.7)
- moved C6 67.3 mm to (131.3, 56.7)
- moved C7 67.3 mm to (135.4, 56.7)
- moved R7 16.8 mm to (56.0, 46.9), turned to 0 degrees
- moved SW1 15.7 mm to (56.0, 54.0), turned to 270 degrees
- moved D33 12.6 mm to (223.5, 68.5)
- moved D34 12.6 mm to (245.0, 68.5)
- moved D39 12.6 mm to (221.2, 87.5)
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Connections:
- K1 pad 1: COL_1 -> Net-(D1-Pad2)
- K1 pad 2: Net-(D1-Pad2) -> COL_1
- K10 pad 1: COL_10 -> Net-(D10-Pad2)
- K10 pad 2: Net-(D10-Pad2) -> COL_10
- K11 pad 1: COL_11 -> Net-(D11-Pad2)
- K11 pad 2: Net-(D11-Pad2) -> COL_11
- K12 pad 1: COL_12 -> Net-(D12-Pad2)
- K12 pad 2: Net-(D12-Pad2) -> COL_12
- K13 pad 1: COL_1 -> Net-(D13-Pad2)
- K13 pad 2: Net-(D13-Pad2) -> COL_1
- K14 pad 1: COL_2 -> Net-(D14-Pad2)
- K14 pad 2: Net-(D14-Pad2) -> COL_2
- K15 pad 1: COL_3 -> Net-(D15-Pad2)
- K15 pad 2: Net-(D15-Pad2) -> COL_3
- K16 pad 1: COL_4 -> Net-(D16-Pad2)
- K16 pad 2: Net-(D16-Pad2) -> COL_4
- K17 pad 1: COL_5 -> Net-(D17-Pad2)
- K17 pad 2: Net-(D17-Pad2) -> COL_5
- K18 pad 1: COL_6 -> Net-(D18-Pad2)
- K18 pad 2: Net-(D18-Pad2) -> COL_6
- K19 pad 1: COL_7 -> Net-(D19-Pad2)
- K19 pad 2: Net-(D19-Pad2) -> COL_7
- K2 pad 1: COL_2 -> Net-(D2-Pad2)
- K2 pad 2: Net-(D2-Pad2) -> COL_2
- K20 pad 1: COL_8 -> Net-(D20-Pad2)
- K20 pad 2: Net-(D20-Pad2) -> COL_8
- K21 pad 1: COL_9 -> Net-(D21-Pad2)
- K21 pad 2: Net-(D21-Pad2) -> COL_9
- K22 pad 1: COL_10 -> Net-(D22-Pad2)
- K22 pad 2: Net-(D22-Pad2) -> COL_10
- K23 pad 1: COL_11 -> Net-(D23-Pad2)
- K23 pad 2: Net-(D23-Pad2) -> COL_11
- K24 pad 1: COL_1 -> Net-(D24-Pad2)
- K24 pad 2: Net-(D24-Pad2) -> COL_1
- K25 pad 1: COL_2 -> Net-(D25-Pad2)
- K25 pad 2: Net-(D25-Pad2) -> COL_2
- K26 pad 1: COL_3 -> Net-(D26-Pad2)
- K26 pad 2: Net-(D26-Pad2) -> COL_3
- K27 pad 1: COL_4 -> Net-(D27-Pad2)
- K27 pad 2: Net-(D27-Pad2) -> COL_4
- K28 pad 1: COL_5 -> Net-(D28-Pad2)
- K28 pad 2: Net-(D28-Pad2) -> COL_5
- K29 pad 1: COL_6 -> Net-(D29-Pad2)
- K29 pad 2: Net-(D29-Pad2) -> COL_6
- K3 pad 1: COL_3 -> Net-(D3-Pad2)
- K3 pad 2: Net-(D3-Pad2) -> COL_3
- K30 pad 1: COL_7 -> Net-(D30-Pad2)
- K30 pad 2: Net-(D30-Pad2) -> COL_7
- K31 pad 1: COL_8 -> Net-(D31-Pad2)
- K31 pad 2: Net-(D31-Pad2) -> COL_8
- K32 pad 1: COL_9 -> Net-(D32-Pad2)
- K32 pad 2: Net-(D32-Pad2) -> COL_9
- K33 pad 1: COL_10 -> Net-(D33-Pad2)
- K33 pad 2: Net-(D33-Pad2) -> COL_10
- K33_1 pad 1: COL_10 -> Net-(D33-Pad2)
- K33_1 pad 2: Net-(D33-Pad2) -> COL_10
- K34 pad 1: COL_11 -> Net-(D34-Pad2)
- K34 pad 2: Net-(D34-Pad2) -> COL_11
- K34_1 pad 1: COL_11 -> Net-(D34-Pad2)
- K34_1 pad 2: Net-(D34-Pad2) -> COL_11
- K35 pad 1: COL_1 -> Net-(D35-Pad2)
- K35 pad 2: Net-(D35-Pad2) -> COL_1
- K36 pad 1: COL_2 -> Net-(D36-Pad2)
- K36 pad 2: Net-(D36-Pad2) -> COL_2
- K37 pad 1: COL_3 -> Net-(D37-Pad2)
- K37 pad 2: Net-(D37-Pad2) -> COL_3
- K37_1 pad 1: COL_3 -> Net-(D37-Pad2)
- K37_1 pad 2: Net-(D37-Pad2) -> COL_3
- K38 pad 1: COL_4 -> Net-(D38-Pad2)
- K38 pad 2: Net-(D38-Pad2) -> COL_4
- K38_1 pad 1: COL_4 -> Net-(D38-Pad2)
- K38_1 pad 2: Net-(D38-Pad2) -> COL_4
- K39 pad 1: COL_5 -> Net-(D39-Pad2)
- K39 pad 2: Net-(D39-Pad2) -> COL_5
- K39_1 pad 1: COL_5 -> Net-(D39-Pad2)
- K39_1 pad 2: Net-(D39-Pad2) -> COL_5
- K4 pad 1: COL_4 -> Net-(D4-Pad2)
- K4 pad 2: Net-(D4-Pad2) -> COL_4
- K40 pad 1: COL_6 -> Net-(D40-Pad2)
- K40 pad 2: Net-(D40-Pad2) -> COL_6
- K41 pad 1: COL_7 -> Net-(D41-Pad2)
- K41 pad 2: Net-(D41-Pad2) -> COL_7
- K42 pad 1: COL_8 -> Net-(D42-Pad2)
- K42 pad 2: Net-(D42-Pad2) -> COL_8
- K5 pad 1: COL_5 -> Net-(D5-Pad2)
- K5 pad 2: Net-(D5-Pad2) -> COL_5
- K6 pad 1: COL_6 -> Net-(D6-Pad2)
- K6 pad 2: Net-(D6-Pad2) -> COL_6
- K7 pad 1: COL_7 -> Net-(D7-Pad2)
- K7 pad 2: Net-(D7-Pad2) -> COL_7
- K8 pad 1: COL_8 -> Net-(D8-Pad2)
- K8 pad 2: Net-(D8-Pad2) -> COL_8
- K9 pad 1: COL_9 -> Net-(D9-Pad2)
- K9 pad 2: Net-(D9-Pad2) -> COL_9
Routing:
- net LEDGND: track 0.00 -> 879.6 mm, vias 0 -> 41
- net +3V3: track 0.00 -> 456.6 mm
- net ROW_1: track 0.00 -> 226.0 mm, vias 0 -> 12
- net ROW_4: track 0.00 -> 215.7 mm, vias 0 -> 8
- net ROW_2: track 0.00 -> 214.8 mm, vias 0 -> 11
- net ROW_3: track 0.00 -> 214.8 mm, vias 0 -> 11
- net VBUS: track 0.00 -> 95.6 mm, vias 0 -> 3
- net +BATT: track 0.00 -> 26.2 mm, vias 0 -> 2
- net Net-(D12-Pad2): track 0.00 -> 8.08 mm
- net Net-(D39-Pad2): track 0.00 -> 8.03 mm
- net Net-(D23-Pad2): track 0.00 -> 8.03 mm
- net Net-(D6-Pad2): track 0.00 -> 8.03 mm
- net Net-(D11-Pad2): track 0.00 -> 8.03 mm
- net Net-(D33-Pad2): track 0.00 -> 8.03 mm
- net Net-(D28-Pad2): track 0.00 -> 8.03 mm
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Other:
- net class Default: clearance 0.15 -> 0.13; trace_width 0.15 -> 0.2
- rule trace_clearance: 0.15 -> 0.13
- rule trace_min: 0.15 -> 0.13

Commit message: power routing
Parts:
- moved JST1 114.0 mm to (90.8, 43.2)
- moved C3 99.5 mm to (95.2, 50.8), turned to 0 degrees
- moved U3 96.0 mm to (95.2, 54.6), turned to 270 degrees
- moved DB1 95.3 mm to (95.2, 46.4), turned to 180 degrees
- moved R3 92.8 mm to (95.2, 58.5), turned to 180 degrees
- moved R7 36.7 mm to (20.1, 39.0)
- moved SW1 36.7 mm to (20.1, 46.1)
- moved C5 22.8 mm to (147.6, 39.0)
- moved C6 22.8 mm to (145.6, 39.0)
- moved C7 22.8 mm to (149.7, 39.0)
- moved U2 22.0 mm to (147.2, 35.3)
- moved R6 20.7 mm to (147.2, 32.3)
- moved R4 18.2 mm to (151.2, 52.4)
- moved R5 18.2 mm to (153.6, 52.4)
- moved CR6 0.74 mm to (166.4, 43.5)
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Connections:
- K39 pad 2: COL_5 -> COL_10
- K39_1 pad 2: COL_5 -> COL_10
- K40 pad 2: COL_6 -> COL_11
- K41 pad 2: COL_7 -> COL_9
- K42 pad 2: COL_8 -> COL_7
Routing:
- net +3V3: track 456.6 -> 1092.3 mm, vias 0 -> 16
- net LEDGND: track 879.6 -> 691.6 mm, vias 41 -> 0
- net ROW_4: track 215.7 -> 97.6 mm, vias 8 -> 0
- net COL_11: track 0.00 -> 89.1 mm
- net COL_10: track 0.00 -> 73.8 mm
- net COL_3: track 0.00 -> 67.4 mm
- net COL_2: track 0.00 -> 67.0 mm
- net COL_4: track 0.00 -> 66.0 mm
- net COL_9: track 0.00 -> 64.1 mm
- net COL_7: track 0.00 -> 64.1 mm
- net COL_1: track 0.00 -> 62.1 mm
- net COL_8: track 0.00 -> 44.0 mm
- net COL_5: track 0.00 -> 44.0 mm
- net COL_6: track 0.00 -> 44.0 mm
- net ROW_1: track 226.0 -> 188.7 mm, vias 12 -> 0
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Other:
- net class Default: clearance 0.13 -> 0.15
- rule trace_clearance: 0.13 -> 0.15

Commit message: routing stuck
Parts:
- moved SW1 36.7 mm to (56.0, 53.9)
- moved R7 36.7 mm to (56.0, 46.6)
- moved R9 19.2 mm to (160.4, 120.1)
- moved G3 4.70 mm to (232.1, 56.5)
- moved G2 4.70 mm to (235.0, 52.0)
- moved R8 0.74 mm to (198.4, 84.2)
Routing:
- net /RESET: track 0.00 -> 174.8 mm, vias 0 -> 5
- net COL_2: track 67.0 -> 192.7 mm, vias 0 -> 3
- net COL_12: track 0.00 -> 123.4 mm, vias 0 -> 3
- net RGB: track 0.00 -> 122.9 mm
- net /7_BLE_IRQ: track 0.00 -> 112.8 mm, vias 0 -> 4
- net /4_SWDIO/RST: track 0.00 -> 112.2 mm, vias 0 -> 4
- net /8_BLE_CS: track 0.00 -> 110.4 mm, vias 0 -> 4
- net /MISO: track 0.00 -> 104.3 mm, vias 0 -> 4
- net /SCK: track 0.00 -> 103.9 mm, vias 0 -> 4
- net /MOSI: track 0.00 -> 103.6 mm, vias 0 -> 4
- net COL_11: track 89.1 -> 181.9 mm, vias 0 -> 3
- net ROW_1: track 188.7 -> 272.8 mm, vias 0 -> 4
- net COL_5: track 44.0 -> 122.7 mm, vias 0 -> 3
- net ROW_2: track 200.0 -> 264.7 mm, vias 0 -> 4
- net COL_6: track 44.0 -> 102.4 mm, vias 0 -> 3
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Other:
- net class Default: trace_width 0.2 -> 0.15
- net class power added: clearance 0.15, trace_width 0.2, via_dia 0.6, via_drill 0.3
